File: FinalPcbLayout/FinalPcbLayout.kicad_sch (KiCad schematic)
At the start: 8 parts, among them J1 Conn_01x04_Pin, J2 Serial Out, J3 Conn_01x11_Pin, J5 Conn_02x05_Odd_Even, SW1 SW_Push, U1 ESP32-WROOM-32, U2 CR2013-MI2120

Commit message: MORE PCB
Connections:
- no-connect marks 19 -> 16
Other:
- added sheet Power (power.kicad_sch)
- added sheet usb (usb.kicad_sch)
Changed lines of the file:
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@@
   (junction (at 224.79 104.14) (diameter 0) (color 0 0 0 0)
   )
-  (no_connect (at 266.7 46.99))
-  (no_connect (at 143.51 87.63))
   (no_connect (at 165.1 46.99))
-  (no_connect (at 168.91 50.8))
   (no_connect (at 100.33 140.97))
   (no_connect (at 52.07 74.93))
@@
       )
     )
+  )
+  (sheet (at 198.12 22.86) (size 31.75 19.05) (fields_autoplaced)
+    (stroke (width 0.1524) (type solid))
+    (fill (color 0 0 0 0.0000))
+    (property "Sheetname" "usb" (at 198.12 22.1484 0)
+      (effects (font (size 1.27 1.27)) (justify left bottom))
+    )
+    (property "Sheetfile" "usb.kicad_sch" (at 198.12 42.4946 0)
+      (effects (font (size 1.27 1.27)) (justify left top))
+    )
+    (instances
+      (project "FinalPcbLayout"
+        (path "/9fcc273e-b318-4ade-b4c7-fe4ddbf9d677" (page "2"))
+      )
+    )
+  )
+  (sheet (at 198.12 50.8) (size 31.75 19.05) (fields_autoplaced)
+    (stroke (width 0.1524) (type solid))
+    (fill (color 0 0 0 0.0000))
+    (property "Sheetname" "Power" (at 198.12 50.0884 0)
+      (effects (font (size 1.27 1.27)) (justify left bottom))
+    )
+    (property "Sheetfile" "power.kicad_sch" (at 198.12 70.4346 0)
+      (effects (font (size 1.27 1.27)) (justify left top))
+    )
+    (instances
+      (project "FinalPcbLayout"
+        (path "/9fcc273e-b318-4ade-b4c7-fe4ddbf9d677" (page "3"))
+      )
+    )

Commit message: sound chip done
Parts:
- removed U3: ~, BenchTop:MAX98357 Breakout, symbol BenchTop:MAX98357
- added C12, C13, C14, C15: C, symbol Device:C
- added FB1, FB2: FerriteBead, symbol Device:FerriteBead
- added J6: Conn_01x02_Pin, symbol Connector:Conn_01x02_Pin
- added U2: ~, symbol OSMI-parts:MAX98357
Connections:
- net +5V: now also C12.1, C13.1, U2.3 (GND), U2.7 (VDD), U2.8 (VDD)
- net GND: now also C12.2, C13.2, C14.2, C15.2, U2.11 (GND), U2.15 (GND)
- new net: C15.1, FB1.1, J6.2 (Pin_2)
- new net: FB1.2, U2.9 (OUTP)
- new net: FB2.2, U2.10 (OUTN)
- new net: C14.1, FB2.1, J6.1 (Pin_1)
- new net BCLK: U2.16 (BCLK)
- new net DIN: U2.1 (DIN)
- new net LRCLK: U2.14 (LRCLK)
- new net SD_MODE: U2.4 (SD_MODE)
- no-connect marks 16 -> 15
Other:
- moved on the sheet: U2

Commit message: beep
Parts:
- removed U2: CR2013-MI2120, BenchTop:CR2013-MI2120, symbol BenchTop:CR2013-MI2120
- added J8: Micro_SD_Card, Connector_Card:microSD_HC_Molex_47219-2001, symbol Connector:Micro_SD_Card
Connections:
- net BCLK is gone; now on net IO21: U2.16 (BCLK)
- net DIN is gone; now on net IO17: U2.1 (DIN)
- net LRCLK is gone; now on net IO22: U2.14 (LRCLK)
- net +3.3V: now also J8.4 (VDD)
- net GND: now also J8.6 (VSS), J8.9 (SHIELD)
- net SCLK: now also J8.5 (CLK)
- net Sense_VN: now also U1.5 (SENSOR_VN)
- no-connect marks 15 -> 14
Other:
- moved on the sheet: C12, C13, C14, C15, FB1, FB2, J6, U2
