File: FinalPcbLayout/FinalPcbLayout.kicad_sch (KiCad schematic)
At the start: 21 parts, among them J2 SPI, J4 C1, J5 Conn_02x05_Odd_Even, J6 Conn_01x02_Pin, J7 Display Socket, J8 Micro_SD_Card, SW1 SW_Push, U1 ESP32-WROOM-E

Commit message: Routed UART Bridge
Parts:
- added C25: 22uf, Capacitor_SMD:C_Elec_4x5.4, symbol Device:C_Small
- added C26: 0.1uf, Capacitor_SMD:C_0603_1608Metric, symbol Device:C_Small
- J5: footprint Connector_PinHeader_1.27mm:PinHeader_2x05_P1.27mm_Vertical -> Connector_PinHeader_1.27mm:PinHeader_2x05_P1.27mm_Vertical_SMD
Connections:
- net +3.3V: now also C25.2, C26.1
- net GND: now also C25.1, C26.2
Changed lines of the file:
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@@
   (junction (at 111.76 148.59) (diameter 0) (color 0 0 0 0)
   )
+  (junction (at 77.47 21.59) (diameter 0) (color 0 0 0 0)
+  )
+  (junction (at 62.23 25.4) (diameter 0) (color 0 0 0 0)
+  )
   (junction (at 78.74 85.09) (diameter 0) (color 0 0 0 0)
+  )
+  (junction (at 71.12 21.59) (diameter 0) (color 0 0 0 0)
   )
   (junction (at 104.14 148.59) (diameter 0) (color 0 0 0 0)
@@
     (stroke (width 0) (type default))
   )
+  (wire (pts (xy 62.23 25.4) (xy 64.77 25.4))
+    (stroke (width 0) (type default))
+  )
   (wire (pts (xy 158.75 29.21) (xy 158.75 38.1))
     (stroke (width 0) (type default))
@@
     (stroke (width 0) (type default))
   )
+  (wire (pts (xy 62.23 25.4) (xy 62.23 21.59))
+    (stroke (width 0) (type default))
+  )
   (wire (pts (xy 162.56 29.21) (xy 162.56 30.48))
     (stroke (width 0) (type default))
@@
     (stroke (width 0) (type default))
   )
+  (wire (pts (xy 62.23 21.59) (xy 64.77 21.59))
+    (stroke (width 0) (type default))
+  )
   (wire (pts (xy 154.94 38.1) (xy 158.75 38.1))
     (stroke (width 0) (type default))
@@
     (stroke (width 0) (type default))
   )
-  (wire (pts (xy 77.47 29.21) (xy 77.47 30.48))
-    (stroke (width 0) (type default))
-  )
   (wire (pts (xy 237.49 41.91) (xy 237.49 55.88))
     (stroke (width 0) (type default))
@@
     (stroke (width 0) (type default))
   )
+  (wire (pts (xy 71.12 25.4) (xy 71.12 21.59))
+    (stroke (width 0) (type default))
+  )
   (wire (pts (xy 110.49 45.72) (xy 116.84 45.72))
     (stroke (width 0) (type default))
@@
     (stroke (width 0) (type default))
   )
+  (wire (pts (xy 77.47 21.59) (xy 77.47 30.48))
+    (stroke (width 0) (type default))
+  )
   (wire (pts (xy 247.65 139.7) (xy 243.84 139.7))
     (stroke (width 0) (type default))
@@
     (stroke (width 0) (type default))
   )
+  (wire (pts (xy 69.85 25.4) (xy 71.12 25.4))
+    (stroke (width 0) (type default))
+  )
   (wire (pts (xy 165.1 133.35) (xy 165.1 143.51))
     (stroke (width 0) (type default))
@@
     (stroke (width 0) (type default))
   )
+  (wire (pts (xy 71.12 21.59) (xy 77.47 21.59))
+    (stroke (width 0) (type default))
+  )
   (wire (pts (xy 120.65 137.16) (xy 125.73 137.16))
     (stroke (width 0) (type default))
@@
     (stroke (width 0) (type default))
   )
+  (wire (pts (xy 77.47 20.32) (xy 77.47 21.59))
+    (stroke (width 0) (type default))
+  )
   (wire (pts (xy 120.65 142.24) (xy 125.73 142.24))
     (stroke (width 0) (type default))
@@
   )
   (wire (pts (xy 44.45 40.64) (xy 38.1 40.64))
+    (stroke (width 0) (type default))
+  )
+  (wire (pts (xy 69.85 21.59) (xy 71.12 21.59))
     (stroke (width 0) (type default))
   )
@@
       (effects (font (size 1.27 1.27)))
     )
-    (property "Footprint" "Connector_PinHeader_1.27mm:PinHeader_2x05_P1.27mm_Vertical" (at 248.92 110.49 0)
+    (property "Footprint" "Connector_PinHeader_1.27mm:PinHeader_2x05_P1.27mm_Vertical_SMD" (at 248.92 110.49 0)
       (effects (font (size 1.27 1.27)) hide)
     )
@@
         (path "/9fcc273e-b318-4ade-b4c7-fe4ddbf9d677"
           (reference "J1") (unit 1)
+        )
+      )
+    )
+  )
+  (symbol (lib_id "Device:C_Small") (at 67.31 25.4 270) (unit 1)
+    (in_bom yes) (on_board yes) (dnp no)
+    (property "Reference" "C26" (at 67.31 27.94 90)
+      (effects (font (size 1.27 1.27)))
+    )
+    (property "Value" "0.1uf" (at 67.31 30.48 90)
+      (effects (font (size 1.27 1.27)))
+    )
+    (property "Footprint" "Capacitor_SMD:C_0603_1608Metric" (at 67.31 25.4 0)
+      (effects (font (size 1.27 1.27)) hide)
+    )
+    (property "Datasheet" "~" (at 67.31 25.4 0)
+      (effects (font (size 1.27 1.27)) hide)
+    )
+    (property "digikey_pn" "" (at 67.31 25.4 90)
+      (effects (font (size 1.27 1.27)) hide)
+    )
+    (pin "2")
+    (pin "1")
+    (instances
+      (project "FinalPcbLayout"
+        (path "/9fcc273e-b318-4ade-b4c7-fe4ddbf9d677"
+          (reference "C26") (unit 1)
         )
       )
@@
     )
   )
+  (symbol (lib_id "Device:C_Small") (at 67.31 21.59 90) (unit 1)
+    (in_bom yes) (on_board yes) (dnp no) (fields_autoplaced)
+    (property "Reference" "C25" (at 67.3163 15.24 90)
+      (effects (font (size 1.27 1.27)))
+    )
+    (property "Value" "22uf" (at 67.3163 17.78 90)
+      (effects (font (size 1.27 1.27)))
+    )
+    (property "Footprint" "Capacitor_SMD:C_Elec_4x5.4" (at 67.31 21.59 0)
+      (effects (font (size 1.27 1.27)) hide)
+    )
+    (property "Datasheet" "~" (at 67.31 21.59 0)
+      (effects (font (size 1.27 1.27)) hide)
+    )
+    (property "digikey_pn" "" (at 67.31 21.59 90)
+      (effects (font (size 1.27 1.27)) hide)
+    )
+    (pin "2")
+    (pin "1")
+    (instances
+      (project "FinalPcbLayout"
+        (path "/9fcc273e-b318-4ade-b4c7-fe4ddbf9d677"
+          (reference "C25") (unit 1)
+        )
+      )
+    )
+  )
+  (symbol (lib_id "power:GND") (at 62.23 25.4 0) (unit 1)
+    (in_bom yes) (on_board yes) (dnp no) (fields_autoplaced)
+    (property "Reference" "#PWR014" (at 62.23 31.75 0)
+      (effects (font (size 1.27 1.27)) hide)
+    )
+    (property "Value" "GND" (at 62.23 30.48 0)
+      (effects (font (size 1.27 1.27)))
+    )
+    (property "Footprint" "" (at 62.23 25.4 0)
+      (effects (font (size 1.27 1.27)) hide)
+    )
+    (property "Datasheet" "" (at 62.23 25.4 0)
+      (effects (font (size 1.27 1.27)) hide)
+    )
+    (pin "1")
+    (instances
+      (project "FinalPcbLayout"
+        (path "/9fcc273e-b318-4ade-b4c7-fe4ddbf9d677"
+          (reference "#PWR014") (unit 1)
+        )
+      )
+    )
+  )
   (symbol (lib_id "Connector:Conn_01x14_Socket") (at 176.53 21.59 90) (unit 1)
     (in_bom yes) (on_board yes) (dnp no) (fields_autoplaced)
@@
     )
   )
-  (symbol (lib_id "power:+3.3V") (at 77.47 29.21 0) (unit 1)
+  (symbol (lib_id "power:+3.3V") (at 77.47 20.32 0) (unit 1)
     (in_bom yes) (on_board yes) (dnp no)
-    (property "Reference" "#PWR017" (at 77.47 33.02 0)
-      (effects (font (size 1.27 1.27)) hide)
-    )
-    (property "Value" "+3.3V" (at 77.47 24.13 0)
-      (effects (font (size 1.27 1.27)))
-    )
-    (property "Footprint" "" (at 77.47 29.21 0)
-      (effects (font (size 1.27 1.27)) hide)
-    )
-    (property "Datasheet" "" (at 77.47 29.21 0)
-      (effects (font (size 1.27 1.27)) hide)
-    )
+    (property "Reference" "#PWR017" (at 77.47 24.13 0)
+      (effects (font (size 1.27 1.27)) hide)
+    )
+    (property "Value" "+3.3V" (at 77.47 15.24 0)
+      (effects (font (size 1.27 1.27)))
+    )
+    (property "Footprint" "" (at 77.47 20.32 0)
+      (effects (font (size 1.27 1.27)) hide)
+    )
+    (property "Datasheet" "" (at 77.47 20.32 0)
+      (effects (font (size 1.27 1.27)) hide)
+    )

Commit message: Final Pcb Routed (without headers)
Parts:
- H1, H2, H3, H4: footprint MountingHole:MountingHole_3.2mm_M3 -> MountingHole:MountingHole_2.2mm_M2_Pad
Connections:
- net C1_CS: now also J4.3 (Pin_3); no longer J4.2 (Pin_2)
- net C1_Limit: now also J4.1 (Pin_1); no longer J4.3 (Pin_3)
- net C1_PWM: now also J4.2 (Pin_2); no longer J4.1 (Pin_1)
Changed lines of the file:
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@@
+    (stroke (width 0) (type default))
+  )
+  (wire (pts (xy 110.49 53.34) (xy 116.84 53.34))
+    (stroke (width 0) (type default))
+  )
+  (wire (pts (xy 124.46 153.67) (xy 124.46 156.21))
+    (stroke (width 0) (type default))
+  )
+  (wire (pts (xy 120.65 153.67) (xy 124.46 153.67))
+    (stroke (width 0) (type default))
+  )
+  (wire (pts (xy 24.13 157.48) (xy 33.02 157.48))
+    (stroke (width 0) (type default))
+  )
+  (wire (pts (xy 176.53 130.81) (xy 176.53 143.51))
     (stroke (width 0) (type default))
   )
@@
     (stroke (width 0) (type default))
   )
-  (wire (pts (xy 110.49 53.34) (xy 116.84 53.34))
-    (stroke (width 0) (type default))
-  )
-  (wire (pts (xy 124.46 153.67) (xy 124.46 156.21))
-    (stroke (width 0) (type default))
-  )
-  (wire (pts (xy 120.65 153.67) (xy 124.46 153.67))
-    (stroke (width 0) (type default))
-  )
-  (wire (pts (xy 24.13 157.48) (xy 33.02 157.48))
-    (stroke (width 0) (type default))
-  )
-  (wire (pts (xy 176.53 130.81) (xy 176.53 143.51))
-    (stroke (width 0) (type default))
-  )
   (wire (pts (xy 120.65 139.7) (xy 125.73 139.7))
     (stroke (width 0) (type default))
@@
     (stroke (width 0) (type default))
   )
+  (wire (pts (xy 250.19 157.48) (xy 254 157.48))
+    (stroke (width 0) (type default))
+  )
   (wire (pts (xy 71.12 85.09) (xy 77.47 85.09))
     (stroke (width 0) (type default))
@@
     (stroke (width 0) (type default))
   )
+  (wire (pts (xy 250.19 162.56) (xy 254 162.56))
+    (stroke (width 0) (type default))
+  )
   (wire (pts (xy 124.46 153.67) (xy 125.73 153.67))
     (stroke (width 0) (type default))
@@
     (stroke (width 0) (type default))
   )
-  (wire (pts (xy 250.19 162.56) (xy 254 162.56))
-    (stroke (width 0) (type default))
-  )
   (wire (pts (xy 162.56 29.21) (xy 163.83 29.21))
     (stroke (width 0) (type default))
@@
   )
   (wire (pts (xy 256.54 107.95) (xy 257.81 107.95))
-    (stroke (width 0) (type default))
-  )
-  (wire (pts (xy 250.19 157.48) (xy 254 157.48))
     (stroke (width 0) (type default))
   )
@@
     (effects (font (size 1.27 1.27)) (justify right bottom))
   )
-  (label "C1_Limit" (at 250.19 162.56 180) (fields_autoplaced)
-    (effects (font (size 1.27 1.27)) (justify right bottom))
-  )
   (label "IO21" (at 120.65 137.16 0) (fields_autoplaced)
     (effects (font (size 1.27 1.27)) (justify left bottom))
@@
     (effects (font (size 1.27 1.27)) (justify right bottom))
   )
+  (label "C1_PWM" (at 250.19 160.02 180) (fields_autoplaced)
+    (effects (font (size 1.27 1.27)) (justify right bottom))
+  )
   (label "TXD" (at 114.3 38.1 0) (fields_autoplaced)
     (effects (font (size 1.27 1.27)) (justify left bottom))
@@
     (effects (font (size 1.27 1.27)) (justify right bottom))
   )
-  (label "C1_CS" (at 250.19 160.02 180) (fields_autoplaced)
-    (effects (font (size 1.27 1.27)) (justify right bottom))
-  )
   (label "SCLK" (at 30.48 154.94 180) (fields_autoplaced)
     (effects (font (size 1.27 1.27)) (justify right bottom))
@@
     (effects (font (size 1.27 1.27)) (justify right bottom))
   )
+  (label "C1_Limit" (at 250.19 157.48 180) (fields_autoplaced)
+    (effects (font (size 1.27 1.27)) (justify right bottom))
+  )
   (label "COPI" (at 243.84 134.62 0) (fields_autoplaced)
     (effects (font (size 1.27 1.27)) (justify left bottom))
@@
     (effects (font (size 1.27 1.27)) (justify right bottom))
   )
-  (label "C1_PWM" (at 250.19 157.48 180) (fields_autoplaced)
-    (effects (font (size 1.27 1.27)) (justify right bottom))
-  )
   (label "ESP_EN" (at 238.76 30.48 180) (fields_autoplaced)
     (effects (font (size 1.27 1.27)) (justify right bottom))
@@
     (effects (font (size 1.27 1.27)) (justify right bottom))
   )
+  (label "C1_CS" (at 250.19 162.56 180) (fields_autoplaced)
+    (effects (font (size 1.27 1.27)) (justify right bottom))
+  )
   (label "IO22" (at 113.03 66.04 0) (fields_autoplaced)
     (effects (font (size 1.27 1.27)) (justify left bottom))
@@
       (effects (font (size 1.27 1.27)) (justify left))
     )
-    (property "Footprint" "MountingHole:MountingHole_3.2mm_M3" (at 142.24 193.04 0)
+    (property "Footprint" "MountingHole:MountingHole_2.2mm_M2_Pad" (at 142.24 193.04 0)
       (effects (font (size 1.27 1.27)) hide)
     )
@@
     )
     (pin "1")
+    (pin "2")
     (pin "3")
-    (pin "2")
     (instances
       (project "FinalPcbLayout"
@@
       (effects (font (size 1.27 1.27)) hide)
     )
+    (pin "1")
     (pin "2")
-    (pin "1")
     (instances
       (project "FinalPcbLayout"
@@
       (effects (font (size 1.27 1.27)) (justify left))
     )
-    (property "Footprint" "MountingHole:MountingHole_3.2mm_M3" (at 151.13 193.04 0)
+    (property "Footprint" "MountingHole:MountingHole_2.2mm_M2_Pad" (at 151.13 193.04 0)
       (effects (font (size 1.27 1.27)) hide)
     )
@@
       (effects (font (size 1.27 1.27)) hide)
     )
-    (pin "4")
+    (pin "1")
     (pin "10")
-    (pin "6")
+    (pin "11")
+    (pin "12")
+    (pin "13")
+    (pin "14")
+    (pin "15")
+    (pin "16")
+    (pin "2")
+    (pin "23")
+    (pin "24")
+    (pin "25")
+    (pin "26")
+    (pin "27")
+    (pin "28")
     (pin "29")
-    (pin "35")
-    (pin "2")
-    (pin "38")
-    (pin "13")
-    (pin "33")
-    (pin "9")
-    (pin "15")
-    (pin "12")
-    (pin "11")
     (pin "3")
-    (pin "27")
     (pin "30")
     (pin "31")
+    (pin "33")
+    (pin "34")
+    (pin "35")
+    (pin "36")
     (pin "37")
+    (pin "38")
+    (pin "39")
+    (pin "4")
     (pin "5")
+    (pin "6")
     (pin "7")
     (pin "8")
-    (pin "14")
-    (pin "1")
-    (pin "24")
-    (pin "16")
-    (pin "28")
-    (pin "25")
-    (pin "23")
-    (pin "34")
-    (pin "36")
-    (pin "39")
-    (pin "26")
+    (pin "9")
     (instances
       (project "FinalPcbLayout"
@@
       (effects (font (size 1.27 1.27)) hide)
     )
+    (pin "1")
     (pin "2")
-    (pin "1")
     (instances
       (project "FinalPcbLayout"
@@
       (effects (font (size 1.27 1.27)) hide)
     )
+    (pin "1")
+    (pin "10")
+    (pin "11")
+    (pin "12")
     (pin "13")
+    (pin "14")
     (pin "2")
-    (pin "8")
-    (pin "12")
-    (pin "6")
-    (pin "14")
-    (pin "1")
-    (pin "5")
     (pin "3")
     (pin "4")
-    (pin "10")
+    (pin "5")
+    (pin "6")
     (pin "7")
-    (pin "11")
+    (pin "8")
     (pin "9")
     (instances
@@
       (effects (font (size 1.27 1.27)) hide)
     )
+    (pin "1")
     (pin "2")
-    (pin "1")
     (instances
       (project "FinalPcbLayout"
@@
     )
     (pin "1")
+    (pin "2")
     (pin "3")
-    (pin "2")
     (instances
       (project "FinalPcbLayout"
@@
       (effects (font (size 1.27 1.27)) (justify left))
     )
-    (property "Footprint" "MountingHole:MountingHole_3.2mm_M3" (at 160.02 193.04 0)
+    (property "Footprint" "MountingHole:MountingHole_2.2mm_M2_Pad" (at 160.02 193.04 0)
       (effects (font (size 1.27 1.27)) hide)
     )
@@
       (effects (font (size 1.27 1.27)) (justify left))
     )
-    (property "Footprint" "MountingHole:MountingHole_3.2mm_M3" (at 168.91 193.04 0)
-      (effects (font (size 1.27 1.27)) hide)
-    )
+    (property "Footprint" "MountingHole:MountingHole_2.2mm_M2_Pad" (at 168.91 193.04 0)
+      (effects (font (size 1.27 1.27)) hide)
+    )
