File: FinalPcbLayout/power.kicad_sch (KiCad schematic)
At the start: 23 parts, among them Q1 NMOS, U4 AMS1117-3.3

Commit message: beep
Parts:
- added C16, C18: 10uF, symbol Device:C
- added C17: 100nF, symbol Device:C
- added C19: 47uF, symbol Device:C
- added L2: L, symbol Device:L
- added R10: 523k, symbol Device:R
- added R11, R12: 100k, symbol Device:R
- added R13: 10k, symbol Device:R
- added U3: ~, symbol OSMI-parts:TPS63070RNM
Connections:
- net +5V: now also C1.2, C9.2, L1.1, U5.1 (BIAS), U5.12 (UVLO_), C18.1, C19.1, R10.1, R12.1, U3.7 (VOUT), U3.8 (VOUT)
- net GND: now also C16.2, C17.2, C18.2, C19.2, R11.2, U3.10 (PGND), U3.4 (GND), U3.6 (FB2)
- net USB_Vin: now also C16.1, R13.1, U3.1 (PS/SYNC), U3.12 (VIN), U3.13 (VIN); no longer C1.2, C9.2, L1.1, U5.1 (BIAS), U5.12 (UVLO_)
- new net: R13.2, U3.14 (EN)
- new net: R10.2, R11.1, U3.5 (FB)
- new net: L2.1, U3.11 (L1)
- new net: L2.2, U3.9 (L2)
- new net: R12.2, U3.2 (PG)
- new net: C17.1, U3.3 (VAUX)

Commit message: broski
Parts:
- C1, C10, C16, C17, C18, C19, C2, C3, C4, C5, C6, C7, C9: footprint (none) -> Capacitor_SMD:C_0201_0603Metric
- D1: footprint (none) -> Diode_SMD:D_0201_0603Metric
- L1, L2: footprint (none) -> Inductor_SMD:L_0201_0603Metric
- Q1: footprint (none) -> Package_SON:WSON-8-1EP_2x2mm_P0.5mm_EP0.9x1.6mm
- R1, R11, R2, R3, R4, R5, R6, R7: footprint (none) -> Resistor_SMD:R_0201_0603Metric
Changed lines of the file:
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@@
       (effects (font (size 1.27 1.27)) (justify right))
     )
-    (property "Footprint" "" (at 76.5048 63.5 0)
+    (property "Footprint" "Capacitor_SMD:C_0201_0603Metric" (at 76.5048 63.5 0)
       (effects (font (size 1.27 1.27)) hide)
     )
@@
       (effects (font (size 1.27 1.27)) (justify right))
     )
-    (property "Footprint" "" (at 120.904 97.536 90)
+    (property "Footprint" "Resistor_SMD:R_0201_0603Metric" (at 120.904 97.536 90)
       (effects (font (size 1.27 1.27)) hide)
     )
@@
       (effects (font (size 1.27 1.27)))
     )
-    (property "Footprint" "" (at 156.21 43.18 0)
+    (property "Footprint" "Inductor_SMD:L_0201_0603Metric" (at 156.21 43.18 0)
       (effects (font (size 1.27 1.27)) hide)
     )
@@
       (effects (font (size 1.27 1.27)))
     )
-    (property "Footprint" "" (at 210.82 43.18 0)
+    (property "Footprint" "Diode_SMD:D_0201_0603Metric" (at 210.82 43.18 0)
       (effects (font (size 1.27 1.27)) hide)
     )
@@
       (effects (font (size 1.27 1.27)) (justify right))
     )
-    (property "Footprint" "" (at 237.7948 88.9 0)
+    (property "Footprint" "Capacitor_SMD:C_0201_0603Metric" (at 237.7948 88.9 0)
       (effects (font (size 1.27 1.27)) hide)
     )
@@
       (effects (font (size 1.27 1.27)) (justify right))
     )
-    (property "Footprint" "" (at 94.2848 93.98 0)
+    (property "Footprint" "Capacitor_SMD:C_0201_0603Metric" (at 94.2848 93.98 0)
       (effects (font (size 1.27 1.27)) hide)
     )
@@
       (effects (font (size 1.27 1.27)) (justify right))
     )
-    (property "Footprint" "" (at 197.104 92.456 90)
+    (property "Footprint" "Resistor_SMD:R_0201_0603Metric" (at 197.104 92.456 90)
       (effects (font (size 1.27 1.27)) hide)
     )
@@
       (effects (font (size 1.27 1.27)))
     )
-    (property "Footprint" "" (at 181.356 72.136 90)
+    (property "Footprint" "Resistor_SMD:R_0201_0603Metric" (at 181.356 72.136 90)
       (effects (font (size 1.27 1.27)) hide)
     )
@@
       (effects (font (size 1.27 1.27)) (justify right))
     )
-    (property "Footprint" "" (at 82.804 91.186 90)
+    (property "Footprint" "Resistor_SMD:R_0201_0603Metric" (at 82.804 91.186 90)
       (effects (font (size 1.27 1.27)) hide)
     )
@@
       (effects (font (size 1.27 1.27)) (justify right))
     )
-    (property "Footprint" "" (at 212.3948 63.5 0)
+    (property "Footprint" "Capacitor_SMD:C_0201_0603Metric" (at 212.3948 63.5 0)
       (effects (font (size 1.27 1.27)) hide)
     )
@@
       (effects (font (size 1.27 1.27)) (justify left))
     )
-    (property "Footprint" "" (at 126.6952 144.78 0)
+    (property "Footprint" "Capacitor_SMD:C_0201_0603Metric" (at 126.6952 144.78 0)
       (effects (font (size 1.27 1.27)) hide)
     )
@@
       (effects (font (size 1.27 1.27)) (justify left))
     )
-    (property "Footprint" "" (at 205.232 144.78 90)
+    (property "Footprint" "Resistor_SMD:R_0201_0603Metric" (at 205.232 144.78 90)
       (effects (font (size 1.27 1.27)) hide)
     )
@@
       (effects (font (size 1.27 1.27)) (justify left))
     )
-    (property "Footprint" "" (at 260.0452 140.97 0)
+    (property "Footprint" "Capacitor_SMD:C_0201_0603Metric" (at 260.0452 140.97 0)
       (effects (font (size 1.27 1.27)) hide)
     )
@@
       (effects (font (size 1.27 1.27)) (justify right))
     )
-    (property "Footprint" "" (at 106.9848 93.98 0)
+    (property "Footprint" "Capacitor_SMD:C_0201_0603Metric" (at 106.9848 93.98 0)
       (effects (font (size 1.27 1.27)) hide)
     )
@@
       (effects (font (size 1.27 1.27)))
     )
-    (property "Footprint" "" (at 162.306 72.136 90)
+    (property "Footprint" "Resistor_SMD:R_0201_0603Metric" (at 162.306 72.136 90)
       (effects (font (size 1.27 1.27)) hide)
     )
@@
       (effects (font (size 1.27 1.27)) (justify left))
     )
-    (property "Footprint" "" (at 242.2652 140.97 0)
+    (property "Footprint" "Capacitor_SMD:C_0201_0603Metric" (at 242.2652 140.97 0)
       (effects (font (size 1.27 1.27)) hide)
     )
@@
       (effects (font (size 1.27 1.27)))
     )
-    (property "Footprint" "" (at 175.26 115.57 0)
+    (property "Footprint" "Inductor_SMD:L_0201_0603Metric" (at 175.26 115.57 0)
       (effects (font (size 1.27 1.27)) hide)
     )
@@
       (effects (font (size 1.27 1.27)) (justify right))
     )
-    (property "Footprint" "" (at 171.7548 90.17 0)
+    (property "Footprint" "Capacitor_SMD:C_0201_0603Metric" (at 171.7548 90.17 0)
       (effects (font (size 1.27 1.27)) hide)
     )
@@
       (effects (font (size 1.27 1.27)) (justify right))
     )
-    (property "Footprint" "" (at 223.774 93.726 90)
+    (property "Footprint" "Resistor_SMD:R_0201_0603Metric" (at 223.774 93.726 90)
       (effects (font (size 1.27 1.27)) hide)
     )
@@
       (effects (font (size 1.27 1.27)) (justify left))
     )
-    (property "Footprint" "" (at 200.66 49.53 0)
+    (property "Footprint" "Package_SON:WSON-8-1EP_2x2mm_P0.5mm_EP0.9x1.6mm" (at 200.66 49.53 0)
       (effects (font (size 1.27 1.27)) hide)
     )
@@
       (effects (font (size 1.27 1.27)) (justify left))
     )
-    (property "Footprint" "" (at 149.5552 148.59 0)
+    (property "Footprint" "Capacitor_SMD:C_0201_0603Metric" (at 149.5552 148.59 0)
       (effects (font (size 1.27 1.27)) hide)
     )
@@
       (effects (font (size 1.27 1.27)) (justify left))
     )
-    (property "Footprint" "" (at 65.7352 152.4 0)
+    (property "Footprint" "Capacitor_SMD:C_0201_0603Metric" (at 65.7352 152.4 0)
       (effects (font (size 1.27 1.27)) hide)
     )
@@
       (effects (font (size 1.27 1.27)) (justify right))
     )
-    (property "Footprint" "" (at 223.774 61.976 90)
+    (property "Footprint" "Resistor_SMD:R_0201_0603Metric" (at 223.774 61.976 90)
       (effects (font (size 1.27 1.27)) hide)
     )
@@
       (effects (font (size 1.27 1.27)) (justify right))
     )
-    (property "Footprint" "" (at 120.9548 86.36 0)
+    (property "Footprint" "Capacitor_SMD:C_0201_0603Metric" (at 120.9548 86.36 0)
       (effects (font (size 1.27 1.27)) hide)
     )
@@
       (effects (font (size 1.27 1.27)) (justify right))
     )
-    (property "Footprint" "" (at 68.8848 82.55 0)
-      (effects (font (size 1.27 1.27)) hide)
-    )
+    (property "Footprint" "Capacitor_SMD:C_0201_0603Metric" (at 68.8848 82.55 0)
+      (effects (font (size 1.27 1.27)) hide)
+    )

Commit message: for jake
Parts:
- U3: footprint (none) -> OSMI-parts:VQFN-15-1EP-2.5x3mm_P0.5mm
Changed lines of the file:
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@@
       (effects (font (size 1.27 1.27)))
     )
-    (property "Footprint" "" (at 175.26 137.16 0)
+    (property "Footprint" "OSMI-parts:VQFN-15-1EP-2.5x3mm_P0.5mm" (at 175.26 137.16 0)
       (effects (font (size 1.27 1.27)) hide)
     )
