File: FinalPcbLayout/usb.kicad_sch (KiCad schematic)
At the start: 26 parts, among them J5 USB_C_Receptacle, Q2 NPN, Q3 NPN, U7 93LCxxB, Y1 12Mhz

Commit message: Sim Disabled
Parts:
- C20, C21, C22, C23, C24, D2, D3, J5, Q2, Q3, R14, R15, R16, R17, R18, R19, R20, R21, R22, R26, R27, R28, R9, U7, Y1: Cost (none) -> 0
- U6: Cost 3.85 -> 0
Changed lines of the file:
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@@
+      (effects (font (size 1.27 1.27)) hide)
+    )
+    (property "Cost" "0" (at 48.26 127 0)
+      (effects (font (size 1.27 1.27)) hide)
+    )
+    (property "Sim.Enable" "0" (at 48.26 127 0)
       (effects (font (size 1.27 1.27)) hide)
     )
@@
       (effects (font (size 1.27 1.27)) hide)
     )
+    (property "Cost" "0" (at 74.93 105.41 0)
+      (effects (font (size 1.27 1.27)) hide)
+    )
+    (property "Sim.Enable" "0" (at 74.93 105.41 0)
+      (effects (font (size 1.27 1.27)) hide)
+    )
     (pin "2")
     (pin "1")
@@
       (effects (font (size 1.27 1.27)) hide)
     )
+    (property "Cost" "0" (at 59.69 110.49 0)
+      (effects (font (size 1.27 1.27)) hide)
+    )
+    (property "Sim.Enable" "0" (at 59.69 110.49 0)
+      (effects (font (size 1.27 1.27)) hide)
+    )
     (pin "2")
     (pin "1")
@@
       (effects (font (size 1.27 1.27)) hide)
     )
+    (property "Cost" "0" (at 95.25 35.56 0)
+      (effects (font (size 1.27 1.27)) hide)
+    )
+    (property "Sim.Enable" "0" (at 95.25 35.56 0)
+      (effects (font (size 1.27 1.27)) hide)
+    )
     (pin "2")
     (pin "1")
@@
     )
     (property "Datasheet" "~" (at 48.26 137.16 0)
+      (effects (font (size 1.27 1.27)) hide)
+    )
+    (property "Cost" "0" (at 48.26 137.16 0)
+      (effects (font (size 1.27 1.27)) hide)
+    )
+    (property "Sim.Enable" "0" (at 48.26 137.16 0)
       (effects (font (size 1.27 1.27)) hide)
     )
@@
     )
     (property "Datasheet" "~" (at 149.86 143.51 0)
+      (effects (font (size 1.27 1.27)) hide)
+    )
+    (property "Cost" "0" (at 149.86 143.51 0)
+      (effects (font (size 1.27 1.27)) hide)
+    )
+    (property "Sim.Enable" "0" (at 149.86 143.51 0)
       (effects (font (size 1.27 1.27)) hide)
     )
@@
       (effects (font (size 1.27 1.27)) hide)
     )
+    (property "Cost" "0" (at 139.7 177.8 0)
+      (effects (font (size 1.27 1.27)) hide)
+    )
+    (property "Sim.Enable" "0" (at 139.7 177.8 0)
+      (effects (font (size 1.27 1.27)) hide)
+    )
     (pin "1")
     (pin "2")
@@
       (effects (font (size 1.27 1.27)) hide)
     )
+    (property "Cost" "0" (at 83.82 35.56 0)
+      (effects (font (size 1.27 1.27)) hide)
+    )
+    (property "Sim.Enable" "0" (at 83.82 35.56 0)
+      (effects (font (size 1.27 1.27)) hide)
+    )
     (pin "2")
     (pin "1")
@@
       (effects (font (size 1.27 1.27)) hide)
     )
+    (property "Cost" "0" (at 254 45.72 0)
+      (effects (font (size 1.27 1.27)) hide)
+    )
+    (property "Sim.Enable" "0" (at 254 45.72 0)
+      (effects (font (size 1.27 1.27)) hide)
+    )
     (pin "1")
     (pin "2")
@@
     )
     (property "Datasheet" "~" (at 149.86 132.08 0)
+      (effects (font (size 1.27 1.27)) hide)
+    )
+    (property "Cost" "0" (at 149.86 132.08 0)
+      (effects (font (size 1.27 1.27)) hide)
+    )
+    (property "Sim.Enable" "0" (at 149.86 132.08 0)
       (effects (font (size 1.27 1.27)) hide)
     )
@@
       (effects (font (size 1.27 1.27)) hide)
     )
+    (property "Cost" "0" (at 139.7 132.08 0)
+      (effects (font (size 1.27 1.27)) hide)
+    )
+    (property "Sim.Enable" "0" (at 139.7 132.08 0)
+      (effects (font (size 1.27 1.27)) hide)
+    )
     (pin "1")
     (pin "2")
@@
       (effects (font (size 1.27 1.27)) hide)
     )
+    (property "Cost" "0" (at 238.76 41.91 0)
+      (effects (font (size 1.27 1.27)) hide)
+    )
+    (property "Sim.Enable" "0" (at 238.76 41.91 0)
+      (effects (font (size 1.27 1.27)) hide)
+    )
     (pin "5")
     (pin "7")
@@
     )
     (property "Datasheet" "~" (at 67.31 107.95 0)
+      (effects (font (size 1.27 1.27)) hide)
+    )
+    (property "Cost" "0" (at 67.31 107.95 0)
+      (effects (font (size 1.27 1.27)) hide)
+    )
+    (property "Sim.Enable" "0" (at 67.31 107.95 0)
       (effects (font (size 1.27 1.27)) hide)
     )
@@
       (effects (font (size 1.27 1.27)) hide)
     )
+    (property "Cost" "0" (at 72.39 152.4 0)
+      (effects (font (size 1.27 1.27)) hide)
+    )
+    (property "Sim.Enable" "0" (at 72.39 152.4 0)
+      (effects (font (size 1.27 1.27)) hide)
+    )
     (pin "1")
     (pin "2")
@@
       (effects (font (size 1.27 1.27)) hide)
     )
+    (property "Cost" "0" (at 226.06 116.84 0)
+      (effects (font (size 1.27 1.27)) hide)
+    )
+    (property "Sim.Enable" "0" (at 226.06 116.84 0)
+      (effects (font (size 1.27 1.27)) hide)
+    )
     (pin "1")
     (pin "2")
@@
     )
     (property "Datasheet" "~" (at 226.06 142.24 0)
+      (effects (font (size 1.27 1.27)) hide)
+    )
+    (property "Cost" "0" (at 226.06 142.24 0)
+      (effects (font (size 1.27 1.27)) hide)
+    )
+    (property "Sim.Enable" "0" (at 226.06 142.24 0)
       (effects (font (size 1.27 1.27)) hide)
     )
@@
       (effects (font (size 1.27 1.27)) hide)
     )
+    (property "Cost" "0" (at 139.7 143.51 0)
+      (effects (font (size 1.27 1.27)) hide)
+    )
+    (property "Sim.Enable" "0" (at 139.7 143.51 0)
+      (effects (font (size 1.27 1.27)) hide)
+    )
     (pin "1")
     (pin "2")
@@
       (effects (font (size 1.27 1.27)) hide)
     )
-    (property "Cost" "3.85" (at 107.95 140.97 0)
+    (property "Cost" "0" (at 107.95 140.97 0)
       (effects (font (size 1.27 1.27)) hide)
     )
     (property "Order-Link" "https://www.digikey.com/en/products/detail/ftdi-future-technology-devices-international-ltd/FT232HPQ-TRAY/13981014" (at 107.95 100.33 0)
+      (effects (font (size 1.27 1.27)) hide)
+    )
+    (property "Sim.Enable" "0" (at 107.95 142.24 0)
       (effects (font (size 1.27 1.27)) hide)
     )
@@
       (effects (font (size 1.27 1.27)) hide)
     )
+    (property "Cost" "0" (at 48.26 132.08 0)
+      (effects (font (size 1.27 1.27)) hide)
+    )
+    (property "Sim.Enable" "0" (at 48.26 132.08 0)
+      (effects (font (size 1.27 1.27)) hide)
+    )
     (pin "2")
     (pin "1")
@@
     )
     (property "cost" ".068" (at 238.76 116.84 0)
+      (effects (font (size 1.27 1.27)) hide)
+    )
+    (property "Cost" "0" (at 238.76 116.84 0)
+      (effects (font (size 1.27 1.27)) hide)
+    )
+    (property "Sim.Enable" "0" (at 238.76 116.84 0)
       (effects (font (size 1.27 1.27)) hide)
     )
@@
       (effects (font (size 1.27 1.27)) hide)
     )
+    (property "Cost" "0" (at 238.76 142.24 0)
+      (effects (font (size 1.27 1.27)) hide)
+    )
+    (property "Sim.Enable" "0" (at 238.76 142.24 0)
+      (effects (font (size 1.27 1.27)) hide)
+    )
     (pin "1")
     (pin "2")
@@
     )
     (property "Datasheet" "https://www.usb.org/sites/default/files/documents/usb_type-c.zip" (at 39.37 46.99 0)
+      (effects (font (size 1.27 1.27)) hide)
+    )
+    (property "Cost" "0" (at 35.56 46.99 0)
+      (effects (font (size 1.27 1.27)) hide)
+    )
+    (property "Sim.Enable" "0" (at 35.56 46.99 0)
       (effects (font (size 1.27 1.27)) hide)
     )
@@
       (effects (font (size 1.27 1.27)) hide)
     )
+    (property "Cost" "0" (at 139.7 175.26 0)
+      (effects (font (size 1.27 1.27)) hide)
+    )
+    (property "Sim.Enable" "0" (at 139.7 175.26 0)
+      (effects (font (size 1.27 1.27)) hide)
+    )
     (pin "1")
     (pin "2")
@@
       (effects (font (size 1.27 1.27)) hide)
     )
+    (property "Cost" "0" (at 83.82 25.4 0)
+      (effects (font (size 1.27 1.27)) hide)
+    )
+    (property "Sim.Enable" "0" (at 83.82 25.4 0)
+      (effects (font (size 1.27 1.27)) hide)
+    )
     (pin "1")
     (pin "2")
@@
       (effects (font (size 1.27 1.27)) hide)
     )
+    (property "Cost" "0" (at 227.33 33.02 0)
+      (effects (font (size 1.27 1.27)) hide)
+    )
+    (property "Sim.Enable" "0" (at 227.33 33.02 0)
+      (effects (font (size 1.27 1.27)) hide)
+    )
     (pin "1")
     (pin "2")
@@
       (effects (font (size 1.27 1.27)) hide)
     )
+    (property "Cost" "0" (at 66.04 128.27 0)
+      (effects (font (size 1.27 1.27)) hide)
+    )
+    (property "Sim.Enable" "0" (at 66.04 128.27 0)
+      (effects (font (size 1.27 1.27)) hide)
+    )

Commit message: Added Footprint to NPN Transistors
Parts:
- Q2, Q3: footprint (none) -> Package_TO_SOT_SMD:SOT-23
Changed lines of the file:
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@@
       (effects (font (size 1.27 1.27)) (justify left))
     )
-    (property "Footprint" "" (at 302.26 116.84 0)
+    (property "Footprint" "Package_TO_SOT_SMD:SOT-23" (at 302.26 116.84 0)
       (effects (font (size 1.27 1.27)) hide)
     )
@@
       (effects (font (size 1.27 1.27)) (justify left))
     )
-    (property "Footprint" "" (at 302.26 142.24 0)
+    (property "Footprint" "Package_TO_SOT_SMD:SOT-23" (at 302.26 142.24 0)
       (effects (font (size 1.27 1.27)) hide)
     )

Commit message: No ERC Errors
Parts:
- removed Q2, Q3: NPN, Package_TO_SOT_SMD:SOT-23, symbol Simulation_SPICE:NPN
- added Q2, Q3: S8050, Package_TO_SOT_THT:TO-92_Inline, symbol Transistor_BJT:S8050
- D2: value LED -> BLUE; Cost 0 -> .3; digikey_pn (none) -> 160-1827-6-ND
- D3: footprint LED_SMD:LED_0201_0603Metric -> LED_SMD:LED_0603_1608Metric; Cost 0 -> .26; digikey_pn (none) -> 160-1447-6-ND
- R18: value ??? -> 25
- R19: value 43 -> 65
- R20, R21, R22, R26, R27, R28: footprint (none) -> Resistor_SMD:R_0603_1608Metric
- Y1: footprint (none) -> Crystal:Crystal_SMD_SeikoEpson_FA238-4Pin_3.2x2.5mm
Connections:
- net DTR: now also Q3.1 (E)
- net ESP_EN: now also Q2.3 (C)
- net ESP_IO0_B: now also Q3.3 (C)
- net RTS: now also Q2.1 (E)
- net at R15.2: now also Q2.2 (B)
- net at R14.2: now also Q3.2 (B)
Other:
- note removed: "Update R to match forward i for D2 & D3"

Commit message: Routed UART Bridge
Connections:
- net +3.3V is gone; now on net +3V3: U6.42 (PWRSAV), U6.6 (RESET)
- net OSCO: now reaches C21.2, U6.16 (OSCO), Y1.1
- net OSCI: now reaches C22.1, U6.15 (OSCI), Y1.2
- net ee_pullup: now reaches R22.2, U7.3 (DI)
- net i_ref: now reaches R9.1, U6.50 (REF)
Changed lines of the file:
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@@
+    (stroke (width 0) (type default))
+  )
+  (wire (pts (xy 128.27 101.6) (xy 128.27 106.68))
     (stroke (width 0) (type default))
   )
@@
     (effects (font (size 1.27 1.27)) (justify left bottom))
   )
+  (label "i_ref" (at 71.12 128.27 0) (fields_autoplaced)
+    (effects (font (size 1.27 1.27)) (justify left bottom))
+  )
   (label "TXLED" (at 134.62 147.32 180) (fields_autoplaced)
     (effects (font (size 1.27 1.27)) (justify right bottom))
@@
     (effects (font (size 1.27 1.27)) (justify left bottom))
   )
+  (label "OSCO" (at 57.15 130.81 0) (fields_autoplaced)
+    (effects (font (size 1.27 1.27)) (justify left bottom))
+  )
   (label "EEDATA" (at 88.9 105.41 180) (fields_autoplaced)
     (effects (font (size 1.27 1.27)) (justify right bottom))
@@
     (effects (font (size 1.27 1.27)) (justify left bottom))
   )
+  (label "OSCI" (at 57.15 133.35 0) (fields_autoplaced)
+    (effects (font (size 1.27 1.27)) (justify left bottom))
+  )
   (label "RTS" (at 213.36 142.24 180) (fields_autoplaced)
     (effects (font (size 1.27 1.27)) (justify right bottom))
@@
     (effects (font (size 1.27 1.27)) (justify right bottom))
   )
+  (label "ee_pullup" (at 254 41.91 0) (fields_autoplaced)
+    (effects (font (size 1.27 1.27)) (justify left bottom))
+  )
   (label "PD1_CC2" (at 62.23 29.21 0) (fields_autoplaced)
     (effects (font (size 1.27 1.27)) (justify left bottom))
@@
     )
   )
-  (symbol (lib_id "power:+3V3") (at 128.27 106.68 0) (unit 1)
-    (in_bom yes) (on_board yes) (dnp no) (fields_autoplaced)
-    (property "Reference" "#PWR037" (at 128.27 110.49 0)
-      (effects (font (size 1.27 1.27)) hide)
-    )
-    (property "Value" "+3V3" (at 128.27 101.6 0)
-      (effects (font (size 1.27 1.27)))
-    )
-    (property "Footprint" "" (at 128.27 106.68 0)
-      (effects (font (size 1.27 1.27)) hide)
-    )
-    (property "Datasheet" "" (at 128.27 106.68 0)
+  (symbol (lib_id "power:+3V3") (at 128.27 101.6 0) (unit 1)
+    (in_bom yes) (on_board yes) (dnp no) (fields_autoplaced)
+    (property "Reference" "#PWR037" (at 128.27 105.41 0)
+      (effects (font (size 1.27 1.27)) hide)
+    )
+    (property "Value" "+3V3" (at 128.27 96.52 0)
+      (effects (font (size 1.27 1.27)))
+    )
+    (property "Footprint" "" (at 128.27 101.6 0)
+      (effects (font (size 1.27 1.27)) hide)
+    )
+    (property "Datasheet" "" (at 128.27 101.6 0)
       (effects (font (size 1.27 1.27)) hide)
     )
@@
         (path "/9fcc273e-b318-4ade-b4c7-fe4ddbf9d677/80fb5872-9ff7-41e5-9921-84d432e9852e"
           (reference "R21") (unit 1)
-        )
-      )
-    )
-  )
-  (symbol (lib_id "power:+3.3V") (at 83.82 116.84 0) (unit 1)
-    (in_bom yes) (on_board yes) (dnp no) (fields_autoplaced)
-    (property "Reference" "#PWR014" (at 83.82 120.65 0)
-      (effects (font (size 1.27 1.27)) hide)
-    )
-    (property "Value" "+3.3V" (at 83.82 111.76 0)
-      (effects (font (size 1.27 1.27)))
-    )
-    (property "Footprint" "" (at 83.82 116.84 0)
-      (effects (font (size 1.27 1.27)) hide)
-    )
-    (property "Datasheet" "" (at 83.82 116.84 0)
-      (effects (font (size 1.27 1.27)) hide)
-    )
-    (pin "1")
-    (instances
-      (project "FinalPcbLayout"
-        (path "/9fcc273e-b318-4ade-b4c7-fe4ddbf9d677/80fb5872-9ff7-41e5-9921-84d432e9852e"
-          (reference "#PWR014") (unit 1)
         )
       )
@@
         )
       )
+    )
+  )
+  (symbol (lib_id "power:+3V3") (at 83.82 116.84 0) (unit 1)
+    (in_bom yes) (on_board yes) (dnp no) (fields_autoplaced)
+    (property "Reference" "#PWR06" (at 83.82 120.65 0)
+      (effects (font (size 1.27 1.27)) hide)
+    )
+    (property "Value" "+3V3" (at 83.82 111.76 0)
+      (effects (font (size 1.27 1.27)))
+    )
+    (property "Footprint" "" (at 83.82 116.84 0)
+      (effects (font (size 1.27 1.27)) hide)
+    )
+    (property "Datasheet" "" (at 83.82 116.84 0)
+      (effects (font (size 1.27 1.27)) hide)
+    )
+    (pin "1")
+    (instances
+      (project "FinalPcbLayout"
+        (path "/9fcc273e-b318-4ade-b4c7-fe4ddbf9d677/80fb5872-9ff7-41e5-9921-84d432e9852e"
+          (reference "#PWR06") (unit 1)
+        )
+      )

Commit message: Fixed Resistance
Parts:
- R19: value 65 -> 68
Changed lines of the file:
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@@
       (effects (font (size 1.27 1.27)) (justify left))
     )
-    (property "Value" "65" (at 152.4 133.35 0)
+    (property "Value" "68" (at 152.4 133.35 0)
       (effects (font (size 1.27 1.27)) (justify left))
     )
