File: FinalPcbLayout/FinalPcbLayout.kicad_pcb (KiCad board)
At the start: 4 copper layers, 103 x 50 mm, 88 parts, among them J1 JTAG, J2 3Term, J3 Barrel_Jack, J4 3Term, J5 USB_C_Receptacle, J6 Speaker_Out, J7 Display Socket, J8 Micro_SD_Card, J9 Power Out, Q1 NMOS, Q2 S8050, Q3 S8050, Q4 PMOS, Q5 PMOS, SW1 SW_Push, U1 ESP32-WROOM-E, U2 MAX98357, U3 TPS63070RNMR, U4 LDI1117-3.3H, U5 LM51551DSSR, U6 FT232HPQ, U7 93LCxxB, Y1 12Mhz

Commit message: Working on USB to UART
Parts:
- removed C1, C2: 100nF, Capacitor_SMD:C_0603_1608Metric
- removed C12, C9: 10uF, Capacitor_SMD:C_0805_2012Metric
- removed C13, C24: 0.1uF, Capacitor_SMD:C_0603_1608Metric
- removed C14, C15: 220pF, Capacitor_SMD:C_0603_1608Metric
- removed C20: 3.3u, Capacitor_SMD:C_0603_1608Metric
- removed C21, C22: 18pf, Capacitor_SMD:C_0603_1608Metric
- removed C23: 33nF, Capacitor_SMD:C_0603_1608Metric
- removed C25, C7: 22uF, Capacitor_SMD:C_Elec_4x5.4
- removed C3: 6.8nF, Capacitor_SMD:C_0603_1608Metric
- removed C4: 15nF, Capacitor_SMD:C_1812_4532Metric
- removed C5, C8: 1uF, Capacitor_SMD:C_0603_1608Metric
- removed C6: 1nF, Capacitor_SMD:C_0805_2012Metric
- removed D2: BLUE, LED_SMD:LED_0603_1608Metric
- removed D3: RED, LED_SMD:LED_0603_1608Metric
- removed FB1, FB2: 120 ohm, Resistor_SMD:R_0603_1608Metric
- removed J4: 3Term, TerminalBlock_TE-Connectivity:TerminalBlock_TE_282834-3_1x03_P2.54mm_Horizontal
- removed J6: Speaker_Out, Connector_PinHeader_2.54mm:PinHeader_1x02_P2.54mm_Horizontal
- removed J9: Power Out, Connector_PinHeader_2.54mm:PinHeader_1x03_P2.54mm_Horizontal
- removed L1: 2.2uH, Inductor_SMD:L_Coilcraft_XAL8080-XXX
- removed Q1: NMOS, Package_SON:WSON-8-1EP_2x2mm_P0.5mm_EP0.9x1.6mm
- removed Q5: PMOS, Package_TO_SOT_SMD:Vishay_PowerPAK_SC70-6L_Single
- removed R16, R17: 1k, Resistor_SMD:R_0603_1608Metric
- removed R18: 25, Resistor_SMD:R_0603_1608Metric
- removed R19: 68, Resistor_SMD:R_0603_1608Metric
- removed R20: 100k 1%, Resistor_SMD:R_0603_1608Metric
- removed R21: 15k 1%, Resistor_SMD:R_0603_1608Metric
- removed R22: 2k, Resistor_SMD:R_0603_1608Metric
- removed R26, R27, R28: 10k 1%, Resistor_SMD:R_0603_1608Metric
- removed R3: 12m, Resistor_SMD:R_1206_3216Metric
- removed R4: 487, Resistor_SMD:R_1206_3216Metric
- removed R5: 100, Resistor_SMD:R_0805_2012Metric
- removed R6: 2.49k, Resistor_SMD:R_0603_1608Metric
- removed R7: 27.4k, Resistor_SMD:R_0603_1608Metric
- removed R8: 370k, Resistor_SMD:R_0603_1608Metric
- removed R9: 12k 1%, Resistor_SMD:R_0603_1608Metric
- removed SW1: SW_Push, TerminalBlock_TE-Connectivity:TerminalBlock_TE_282834-2_1x02_P2.54mm_Horizontal
- removed U5: LM51551DSSR, Package_SON:WSON-12-1EP_3x2mm_P0.5mm_EP1x2.65_ThermalVias
- removed U6: FT232HPQ, Package_DFN_QFN:QFN-56-1EP_8x8mm_P0.5mm_EP4.5x5.2mm_ThermalVias
- removed U7: 93LCxxB, Package_SO:SOIC-8_3.9x4.9mm_P1.27mm
- removed Y1: 12Mhz, Crystal:Crystal_SMD_SeikoEpson_FA238-4Pin_3.2x2.5mm
- D1: footprint SL42_E3_57T:CR_2-E3&slash_57T_VIS -> Diode_SMD:D_SMA
- J2: value 3Term -> Conn_01x10
- J7: footprint Connector_PinSocket_2.54mm:PinSocket_1x14_P2.54mm_Vertical -> Connector_PinSocket_2.54mm:PinSocket_1x14_P2.54mm_Vertical_SMD_Pin1Left
- R1: value 3.3k -> 5.1k 20%
- R2: value 21k -> 5.1k 20%
- U2: value MAX98357 -> FT231XQ; footprint Package_DFN_QFN:QFN-16-1EP_3x3mm_P0.5mm_EP1.45x1.45mm -> Package_DFN_QFN:QFN-20-1EP_4x4mm_P0.5mm_EP2.5x2.5mm
- moved Q2 101.9 mm to (55.6, 68.9), turned to 0 degrees
- moved Q3 101.8 mm to (55.6, 74.7), turned to 0 degrees
- moved R14 99.8 mm to (62.2, 71.9), turned to 0 degrees
- moved R15 92.7 mm to (62.2, 74.4), turned to 0 degrees
- moved C11 90.8 mm to (68.0, 55.7), turned to 0 degrees
- moved C10 89.9 mm to (68.2, 52.9), turned to 0 degrees
- moved Q4 82.1 mm to (67.9, 58.9), turned to 0 degrees
- moved J7 76.9 mm to (157.0, 104.9)
- moved J3 72.4 mm to (59.2, 48.9), turned to 0 degrees
- moved R1 61.9 mm to (62.2, 66.9), turned to 0 degrees
- moved R2 46.9 mm to (62.2, 69.4), turned to 0 degrees
- moved D1 46.9 mm to (143.8, 90.9), turned to -90 degrees
- moved J8 34.9 mm to (143.5, 121.7), turned to 0 degrees
- moved U2 30.1 mm to (124.6, 113.6), turned to 0 degrees
- moved U4 17.5 mm to (146.8, 83.6), turned to 0 degrees
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Connections:
- C16 pad 1: /Power/V_in -> +12V
- D1 pad 1: +12V -> /Power/D1-U4
- D1 pad 2: Net-(D1-A) -> +5V
- J2 pad 1: /COPI -> +12V
- J2 pad 2: /CIPO -> /COPI
- J2 pad 3: /SCLK -> /CIPO
- J3 pad 1: Net-(Q5-D) -> +12V
- J5 pad A5: /usb/PD1_CC1 -> Net-(J5-CC1)
- J5 pad B5: /usb/PD1_CC2 -> Net-(J5-CC2)
- Q4 pad 4: /Power/V_in -> +12V
- R1 pad 1: GND -> Net-(J5-CC2)
- R1 pad 2: Net-(C4-Pad1) -> GND
- R13 pad 1: /Power/V_in -> +12V
- R2 pad 1: GND -> Net-(J5-CC1)
- R2 pad 2: Net-(U5-RT) -> GND
- U1 pad 28: /IO17 -> /C1_ENC_P
- U1 pad 33: /IO21 -> /C1_ENC_N
- U1 pad 36: /IO22 -> unconnected-(U1-GPIO22-Pad36)
- U1 pad 7: /SD_CS -> unconnected-(U1-GPIO35/ADC1_CH7-Pad7)
- U1 pad 8: /IO32 -> unconnected-(U1-32K_XP/GPIO32/ADC1_CH4-Pad8)
- U1 pad 9: /IO33 -> /SD_CS
- U2 pad 1: /IO17 -> unconnected-(U2-RXD-Pad1)
- U2 pad 10: Net-(U2-OUTN) -> unconnected-(U2-3V3OUT-Pad10)
- U2 pad 11: GND -> unconnected-(U2-~{RESET}-Pad11)
- U2 pad 12: (no net) -> unconnected-(U2-VCC-Pad12)
- U2 pad 13: (no net) -> unconnected-(U2-GND-Pad13)
- U2 pad 14: /IO22 -> unconnected-(U2-CBUS1-Pad14)
- U2 pad 15: GND -> unconnected-(U2-CBUS0-Pad15)
- U2 pad 16: /IO21 -> unconnected-(U2-CBUS3-Pad16)
- U2 pad 17: (no net) -> unconnected-(U2-TXD-Pad17)
- U2 pad 3: GND -> unconnected-(U2-GND-Pad3)
- U2 pad 4: /SD_MODE -> unconnected-(U2-~{DSR}-Pad4)
- U2 pad 5: (no net) -> unconnected-(U2-~{DCD}-Pad5)
- U2 pad 6: (no net) -> unconnected-(U2-~{CTS}-Pad6)
- U2 pad 7: +5V -> unconnected-(U2-CBUS2-Pad7)
- U2 pad 8: +5V -> unconnected-(U2-USBDP-Pad8)
- U2 pad 9: Net-(U2-OUTP) -> unconnected-(U2-USBDM-Pad9)
- U3 pad 1: /Power/V_in -> +12V
- U3 pad 12: /Power/V_in -> +12V
- U3 pad 13: /Power/V_in -> +12V
- U4 pad 3: +5V -> /Power/D1-U4
Routing:
- net /COPI: track 179.2 -> 0.00 mm, vias 3 -> 0
- net /CIPO: track 161.4 -> 0.00 mm, vias 2 -> 0
- net +3.3V: track 166.7 -> 6.05 mm, vias 2 -> 11
- net /SCLK: track 158.3 -> 0.00 mm, vias 5 -> 0
- net /Power/V_in: track 106.4 -> 0.00 mm, vias 2 -> 0
- net /Touch_CS: track 103.7 -> 0.00 mm, vias 1 -> 0
- net /Display_RST: track 101.9 -> 0.00 mm, vias 2 -> 0
- net /Display_DC: track 101.8 -> 0.00 mm, vias 1 -> 0
- net /Display_CS: track 100.0 -> 0.00 mm, vias 1 -> 0
- net /TXD: track 64.9 -> 0.00 mm, vias 2 -> 0
- net /RXD: track 64.0 -> 0.00 mm, vias 2 -> 0
- net /ESP_EN: track 64.7 -> 3.47 mm, vias 5 -> 0
- net +12V: track 59.4 -> 3.76 mm, vias 3 -> 0
- net +3V3: track 54.7 -> 0.00 mm, vias 14 -> 0
- net /C1_Limit: track 51.6 -> 0.00 mm, vias 2 -> 0
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- added copper zone on In2.Cu, net +3.3V
- added copper zone on B.Cu, net GND
- removed copper zone on F.Cu, net +12V
- removed copper zone on In2.Cu, net +5V
